File: PCB/Classic MIDI FeatherWing.kicad_pcb (KiCad board)
At the start: 2 copper layers, 50.8 x 22.9 mm, 21 parts, among them J1 MIDI_IN, J2 MIDI_OUT, J3 TRS_MIDI_IN, J4 TRS_MIDI_OUT, U1 ICPL0601, U2 74HCT1G125, U3 74HCT1G125, U4 Feather, U5 74HCT1G125

Commit message: update silkscreen
Parts:
- D1: value 1N4001 -> SD0805
